File: Blueprint_PCB_AW_V3.kicad_pcb (KiCad board)
At the start: 2 copper layers, 23 parts, among them J1 Conn_01x04_Pin, SW1 SW_Push, SW10 RotaryEncoder_Switch, SW2 SW_Push, SW3 SW_Push, SW4 SW_Push, SW5 SW_Push, SW6 SW_Push, SW7 SW_Push, SW8 SW_Push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

Commit message: Work on PCB Finish V1
Parts:
- removed J1: Conn_01x04_Pin, Connector:FanPinHeader_1x04_P2.54mm_Vertical
- added J2: Conn_01x04_Pin, Connector_PinHeader_2.54mm:PinHeader_1x04_P2.54mm_Vertical, F.Cu at (154.8, 28.1)
- SW1, SW2, SW3, SW4, SW5, SW6, SW7, SW8, SW9: footprint Button_Switch_THT:SW_PUSH_6mm_H5mm -> Button_Switch_Keyboard:SW_Cherry_MX_1.00u_Plate
- moved SW7 77.0 mm to (156.5, 42.8)
- moved SW8 76.6 mm to (156.5, 57.9)
- moved SW9 76.4 mm to (156.5, 73.0)
- moved SW4 72.5 mm to (141.4, 42.8)
- moved SW5 72.1 mm to (141.4, 57.9)
- moved SW6 71.9 mm to (141.4, 73.0)
- moved SW1 68.0 mm to (126.3, 42.8)
- moved SW2 67.6 mm to (126.3, 57.9)
- moved SW3 67.4 mm to (126.3, 73.0)
- moved SW10 66.9 mm to (165.0, 28.5)
- moved U1 66.2 mm to (138.9, 98.7), turned to 180 degrees
- moved D7 59.4 mm to (104.1, 70.9)
- moved D8 59.4 mm to (104.1, 74.5)
- moved D6 59.2 mm to (104.1, 67.4)
- moved D5 59.1 mm to (104.1, 63.8)
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Connections:
- D1 pad 1: COL2 -> ROW1
- D2 pad 1: COL2 -> ROW2
- D3 pad 1: COL2 -> ROW3
- D7 pad 1: ROW1 -> COL2
- D8 pad 1: ROW2 -> COL2
- D9 pad 1: ROW3 -> COL2
- SW1 pad 1: Net-(D7-A) -> Net-(D1-A)
- SW10 pad A: Net-(C1-Pad2) -> Net-(C2-Pad2)
- SW10 pad B: Net-(C2-Pad2) -> Net-(C1-Pad2)
- SW2 pad 1: Net-(D8-A) -> Net-(D2-A)
- SW3 pad 1: Net-(D6-A) -> Net-(D3-A)
- SW3 pad 2: COL2 -> COL1
- SW4 pad 1: Net-(D5-A) -> Net-(D4-A)
- SW5 pad 1: Net-(D3-A) -> Net-(D5-A)
- SW5 pad 2: COL3 -> COL2
- SW6 pad 1: Net-(D2-A) -> Net-(D6-A)
- SW6 pad 2: COL3 -> COL2
- SW7 pad 1: Net-(D9-A) -> Net-(D7-A)
- SW7 pad 2: COL1 -> COL3
- SW8 pad 1: Net-(D4-A) -> Net-(D8-A)
- SW8 pad 2: COL2 -> COL3
- SW9 pad 1: Net-(D1-A) -> Net-(D9-A)
Routing:
- net GND: track 0.00 -> 134.9 mm
- net COL2: track 0.00 -> 128.6 mm
- net ENC_SW: track 0.00 -> 96.7 mm
- net 3V3: track 0.00 -> 90.0 mm
- net ROW1: track 0.00 -> 79.6 mm
- net Net-(D7-A): track 0.00 -> 71.3 mm
- net SCL: track 0.00 -> 64.8 mm
- net SDA: track 0.00 -> 63.9 mm
- net COL1: track 0.00 -> 59.2 mm
- net Net-(D8-A): track 0.00 -> 58.5 mm
- net ROW2: track 0.00 -> 57.5 mm
- net ROW3: track 0.00 -> 51.4 mm
- net Net-(D9-A): track 0.00 -> 48.8 mm
- net Net-(D4-A): track 0.00 -> 42.9 mm
- net Net-(D6-A): track 0.00 -> 33.4 mm
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