File: Blueprint_PCB_AW_V3.kicad_pcb (KiCad board)
At the start: 2 copper layers, 100 x 100 mm, 37 parts, among them J2 Conn_01x04_Pin, SW1 SW_Push, SW10 SW_Push, SW11 SW_Push, SW12 SW_Push, SW13 SW_Push, SW14 SW_Push, SW15 SW_Push, SW16 SW_Push, SW17 RotaryEncoder_Switch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

Commit message: Few tries to 3D Model absolutly not Finished but PCB is 100 % ready
Parts:
- moved SW17 2.98 mm to (173.8, 24.5)
- moved C1 2.54 mm to (171.8, 36.5)
- moved C2 2.54 mm to (171.8, 39.0)
- moved D10 2.54 mm to (176.3, 66.6)
- moved D11 2.54 mm to (176.3, 70.1)
- moved D12 2.54 mm to (176.3, 73.7)
- moved D13 2.54 mm to (176.3, 77.2)
- moved D14 2.54 mm to (176.3, 80.8)
- moved D15 2.54 mm to (176.3, 84.3)
- moved D16 2.54 mm to (176.3, 87.9)
- moved D9 2.54 mm to (176.3, 63.0)
- moved SW10 2.54 mm to (150.8, 61.6)
- moved SW11 2.54 mm to (150.8, 76.7)
- moved SW12 2.54 mm to (150.8, 91.8)
- moved SW5 2.54 mm to (135.7, 46.5)
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Other:
- outline, holes or cut-outs redrawn
