File: Blueprint_PCB_AW_V3.kicad_sch (KiCad schematic)
At the start: 23 parts, among them J1 Conn_01x04_Pin, SW1 SW_Push, SW10 RotaryEncoder_Switch, SW2 SW_Push, SW3 SW_Push, SW4 SW_Push, SW5 SW_Push, SW6 SW_Push, SW7 SW_Push, SW8 SW_Push, SW9 SW_Push, U1 XIAO-RP2040-DIP

Commit message: Work on PCB Finish V1
Parts:
- removed J1: Conn_01x04_Pin, Connector:FanPinHeader_1x04_P2.54mm_Vertical, symbol Connector:Conn_01x04_Pin
- added J2: Conn_01x04_Pin, Connector_PinHeader_2.54mm:PinHeader_1x04_P2.54mm_Vertical, symbol Connector:Conn_01x04_Pin
- SW1, SW2, SW9: footprint Button_Switch_THT:SW_PUSH_6mm_H5mm -> Button_Switch_Keyboard:SW_Cherry_MX_1.00u_Plate
- SW3: renamed from SW7; footprint Button_Switch_THT:SW_PUSH_6mm_H5mm -> Button_Switch_Keyboard:SW_Cherry_MX_1.00u_Plate
- SW4: renamed from SW3; footprint Button_Switch_THT:SW_PUSH_6mm_H5mm -> Button_Switch_Keyboard:SW_Cherry_MX_1.00u_Plate
- SW5: renamed from SW4; footprint Button_Switch_THT:SW_PUSH_6mm_H5mm -> Button_Switch_Keyboard:SW_Cherry_MX_1.00u_Plate
- SW6: renamed from SW8; footprint Button_Switch_THT:SW_PUSH_6mm_H5mm -> Button_Switch_Keyboard:SW_Cherry_MX_1.00u_Plate
- SW7: renamed from SW5; footprint Button_Switch_THT:SW_PUSH_6mm_H5mm -> Button_Switch_Keyboard:SW_Cherry_MX_1.00u_Plate
- SW8: renamed from SW6; footprint Button_Switch_THT:SW_PUSH_6mm_H5mm -> Button_Switch_Keyboard:SW_Cherry_MX_1.00u_Plate
- renumbered C2 to C1, C1 to C2, D7 to D1, D8 to D2, D9 to D3, D6 to D4, D4 to D6, D3 to D7, D2 to D8, D1 to D9
Connections:
- net 3V3: now also J2.2 (Pin_2)
- net GND: now also J2.1 (Pin_1)
- net SCL: now also J2.3 (Pin_3)
- net SDA: now also J2.4 (Pin_4)

Commit message: Finished PCB
Parts:
- added D12, D13, D14, D15, D16, D4, D8: D, Diode_THT:D_DO-35_SOD27_P7.62mm_Horizontal, symbol Device:D
- added SW12, SW13, SW14, SW15, SW16, SW4, SW8: SW_Push, Button_Switch_Keyboard:SW_Cherry_MX_1.00u_PCB, symbol Switch:SW_Push
- J2: footprint Connector_PinHeader_2.54mm:PinHeader_1x04_P2.54mm_Vertical -> KiCad-SSD1306-0.91-OLED-4pin-128x32.pretty-master:SSD1306-0.91-OLED-4pin-128x32
- SW1, SW2, SW3: footprint Button_Switch_Keyboard:SW_Cherry_MX_1.00u_Plate -> Button_Switch_Keyboard:SW_Cherry_MX_1.00u_PCB
- SW10: renamed from SW8; footprint Button_Switch_Keyboard:SW_Cherry_MX_1.00u_Plate -> Button_Switch_Keyboard:SW_Cherry_MX_1.00u_PCB
- SW11: renamed from SW9; footprint Button_Switch_Keyboard:SW_Cherry_MX_1.00u_Plate -> Button_Switch_Keyboard:SW_Cherry_MX_1.00u_PCB
- SW17: renamed from SW10; footprint Rotary_Encoder:RotaryEncoder_Alps_EC11E-Switch_Vertical_H20mm -> Rotary_Encoder:RotaryEncoder_Alps_EC11E-Switch_Vertical_H20mm_CircularMountingHoles
- SW5: renamed from SW4; footprint Button_Switch_Keyboard:SW_Cherry_MX_1.00u_Plate -> Button_Switch_Keyboard:SW_Cherry_MX_1.00u_PCB
- SW6: renamed from SW5; footprint Button_Switch_Keyboard:SW_Cherry_MX_1.00u_Plate -> Button_Switch_Keyboard:SW_Cherry_MX_1.00u_PCB
- SW7: renamed from SW6; footprint Button_Switch_Keyboard:SW_Cherry_MX_1.00u_Plate -> Button_Switch_Keyboard:SW_Cherry_MX_1.00u_PCB
- SW9: renamed from SW7; footprint Button_Switch_Keyboard:SW_Cherry_MX_1.00u_Plate -> Button_Switch_Keyboard:SW_Cherry_MX_1.00u_PCB
- renumbered D8 to D10, D9 to D11, D4 to D5, D5 to D6, D6 to D7, D7 to D9
Connections:
- net COL1: now also D8.1 (K), SW4.2
- net COL2: now also D12.1 (K), SW8.2
- net COL3: now also D13.1 (K), D14.1 (K), D15.1 (K), D16.1 (K), SW12.2
- net ROW1: now also U1.7 (GPIO0/TX); no longer U1.4 (GPIO29/ADC3/A3)
- net ROW4: now reaches U1.8 (GPIO1/RX)
- net ROW4: now also D4.1 (K)
- new net: D12.2 (A), SW12.1
- new net: D8.2 (A), SW8.1
- new net: D13.2 (A), SW13.1
- new net: D4.2 (A), SW4.1
- new net: D14.2 (A), SW14.1
- new net: D16.2 (A), SW16.1
- new net: D15.2 (A), SW15.1
- new net COL4: SW13.2, SW14.2, SW15.2, SW16.2, U1.4 (GPIO29/ADC3/A3)
- no-connect marks 3 -> 1
Other:
- moved on the sheet: J2
