File: Shematic/Blueprint_PCB_AW_V3.kicad_pcb (KiCad board)
At the start: 2 copper layers, 100 x 100 mm, 37 parts, among them J2 Conn_01x04_Pin, SW1 SW_Push, SW10 SW_Push, SW11 SW_Push, SW12 SW_Push, SW13 SW_Push, SW14 SW_Push, SW15 SW_Push, SW16 SW_Push, SW17 RotaryEncoder_Switch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

Commit message: big changes in Structur Finished Full Case design -> I just have to split it
Other:
- board text added: "Made in Mürztal by wetzi"
- board text removed: "2026"
- board text removed: "Made on earth by wetzi"
Changed lines of the file:
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@@
 		(layer "Edge.Cuts")
 	)
-	(gr_text "2026\n"
+	(gr_text "\n"
 		(at 103.886 108.458 0)
 		(layer "Edge.Cuts")
@@
 		)
 	)
-	(gr_text "Made on earth by wetzi\n\n"
+	(gr_text "Made in Mürztal\nby wetzi"
 		(at 93.5355 112.522 0)
 		(layer "Edge.Cuts")
