File: PCB/Blueprint_PCB_AW_V3.kicad_sch (KiCad schematic)
At the start: 37 parts, among them J2 Conn_01x04_Pin, SW1 SW_Push, SW10 SW_Push, SW11 SW_Push, SW12 SW_Push, SW13 SW_Push, SW14 SW_Push, SW15 SW_Push, SW16 SW_Push, SW17 RotaryEncoder_Switch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

Commit message: big changes I lowkey designed new board
Parts:
- removed D13, D14, D15, D16: D, Diode_THT:D_DO-35_SOD27_P7.62mm_Horizontal, symbol Device:D
- removed SW13, SW14, SW15, SW16: SW_Push, Button_Switch_Keyboard:SW_Cherry_MX_1.00u_PCB, symbol Switch:SW_Push
Connections:
- net COL4: no longer names the net of U1.4 (GPIO29/ADC3/A3)
- no-connect marks 1 -> 2
